Commit message: Update hardware control and MoveIt launch

File: src/dzb_description/urdf/dzb_description.ros2_control.xacro (robot description, xacro)
@@ -2,11 +2,12 @@
 <robot xmlns:xacro="http://www.ros.org/wiki/xacro">
   <xacro:macro name="dzb_description_ros2_control"
-               params="name initial_positions_file use_mock:=true">
+               params="name initial_positions_file use_mock:=false startup_enabled_joints:=pitch_joint">
     <ros2_control name="${name}" type="system">
       <hardware>
         <plugin>motor_control/MotorControlHardwareInterface</plugin>
         <param name="use_mock">${use_mock}</param>
+        <param name="startup_enabled_joints">${startup_enabled_joints}</param>
         <param name="can_channel">0</param>
-        <param name="baud_rate">1000</param>
+        <param name="baud_rate">500</param>
       </hardware>
       <joint name="yaw_joint">

File: src/dzb_description/urdf/dzb_description.urdf.xacro (robot description, xacro)
@@ -2,5 +2,6 @@
 <robot xmlns:xacro="http://www.ros.org/wiki/xacro" name="dzb_description">
     <xacro:arg name="initial_positions_file" default="$(find dzb_moveit_config)/config/initial_positions.yaml" />
-    <xacro:arg name="use_mock" default="true" />
+    <xacro:arg name="use_mock" default="false" />
+    <xacro:arg name="startup_enabled_joints" default="pitch_joint" />
     <!-- Import dzb_description urdf file -->
     <xacro:include filename="$(find dzb_description)/urdf/dzb_robot.urdf" />
@@ -10,4 +11,5 @@
         name="DzbHardwareSystem"
         initial_positions_file="$(arg initial_positions_file)"
-        use_mock="$(arg use_mock)"/>
+        use_mock="$(arg use_mock)"
+        startup_enabled_joints="$(arg startup_enabled_joints)"/>
 </robot>

File: src/dzb_description/urdf/dzb_robot.urdf (robot description, URDF)
Before this commit: robot dzb_description, 6 links, 5 joints
Joints:
- joint trans_joint: limit lower=0.0 upper=0.5 effort=100 velocity=0.2 -> lower=-0.5 upper=0.0 effort=100 velocity=0.2
